File: m5stack_board_dynamixel_ttl_rs3485.kicad_pcb (KiCad board)
At the start: 2 copper layers, 50 x 20 mm, 19 parts, among them J1 B2B-XH-A(LF)(SN), J2 WAFER-HY2.0-4PZZ, J3 B3B-EH-A(LF)(SN), J4 B3B-EH-A(LF)(SN), Q1 2SA1162GR, U1 MAX3485, U2 AP7333-33SAG

Commit message: update board
Parts:
- added JP1: Jumper_2_Open, Jumper:SolderJumper-2_P1.3mm_Open_RoundedPad1.0x1.5mm, B.Cu at (151.5, 111.4)
- moved R1 1.46 mm to (140.8, 121.8)
- moved R2 1.44 mm to (139.9, 120.0)
Connections:
- J2 pad 1: /STS_TX -> /STS_RX
- J2 pad 2: /STS_RX -> /STS_TX
Routing:
- net +5V: track 15.2 -> 21.7 mm
- net /STS_TX: track 17.2 -> 23.0 mm
- net /BAT: track 19.6 -> 24.7 mm
- net Net-(Q1-C): track 13.2 -> 16.1 mm
- net /STS_RX: track 13.0 -> 14.6 mm
- net Net-(Q1-B): track 1.96 -> 3.38 mm
- net GND: vias 26 -> 25
Other:
- board text added: "BAT"
- board text added: "DYNAMIXEL TTL UART Board v2.0 by B-SKY Lab"
- board text added: "G"
- board text added: "GND"
- board text added: "Rx"
- board text added: "Sig"
- board text added: "Tx"
- board text added: "V"
- board text removed: "DYNAMIXEL TTL UART Board v1.0 by B-SKY Lab"
